File: laserboard/RX_AF_sim(standalone).kicad_sch (KiCad schematic)
At the start: 41 parts, among them U1 AD8656 (1/2), U2 AD8656 (1/2 equivalent), U3 AD8656 (1/2 equivalent), U5 AD8656 (1/2 equivalent), U9 AD8656 (1/2)

Commit message: Update
Parts:
- I2: value AC 1 PULSE(0 4u 1n 1n 1n 0.8u 1.6u) -> AC 1 PULSE(0 10u 1n 1n 1n 0.8u 1.6u)
- V1: value 5 -> 3.3
Connections:
- net +5V: no longer C3.2, I2.1, Iambient1.1, Inoise1.1, R3.2, R31.2, R33.2, Rsim2.1, U1.3 (V+), U2.3 (V+), U3.3 (V+), U5.3 (V+)
- new net +3V3: C3.2, I2.1, Iambient1.1, Inoise1.1, R3.2, R31.2, R33.2, Rsim2.1, U1.3 (V+), U2.3 (V+), U3.3 (V+), U5.3 (V+)
Other:
- note added: "Gain control simulation (In real PCB PGA will be used, but it's similar to x1,x2,x4,x8,x16... noninverting amp"
- note removed: "Gain control simulation"
