File: laserboard/laserboard.kicad_sch (KiCad schematic)
At the start: 15 parts, among them U1 AD8656 (1/2 equivalent), U2 AD8656 (1/2 equivalent)

Commit message: Progress backup
Parts:
- added C4, C5: 10p, symbol Device:C
- added C6: 1n, symbol Device:C
- added C7: 330p, symbol Device:C
- added C8: 10uF, symbol Device:C_Polarized
- added I1: ITRNOISE, symbol Simulation_SPICE:ITRNOISE
- added R10: 162, symbol Device:R
- added R11: 487, symbol Device:R
- added R12, R13: 47k, symbol Device:R
- added R2: 8k, symbol Device:R
- added R7: 63.5k, symbol Device:R
- added R8: 360, symbol Device:R
- added R9: 825, symbol Device:R
- added U3, U4: AD8656 (1/2 equivalent), symbol Amplifier_Operational:AD8655
- added V5: 2.5, symbol Simulation_SPICE:VDC
- C3: value 25p -> 30p
- I2: value AC 1 PULSE(0 4u 1n 1n 1n 1u 2u) -> AC 1 PULSE(0 4u 1n 1n 1n 0.5u 1u)
Connections:
- net +5V: now also U1.7 (V+), U2.7 (V+), R13.2, U4.7 (V+)
- net GND: now also C3.1, I2.2, R3.1, U1.4 (V-), U2.4 (V-), C8.2, I1.2, R12.1, U4.4 (V-), V5.2; no longer C2.1, R5.1, U1.3 (+)
- net V+: now also U3.7 (V+); no longer U1.7 (V+), U2.7 (V+)
- net V-: now also U3.4 (V-); no longer U1.4 (V-), U2.4 (V-)
- net Vbias: no longer C3.1, I2.2, R3.1
- net BPW34: now reaches C1.1, C3.2, I2.1, R1.1, R3.2, U1.2 (-)
- net BPW34: now also I1.1
- net OPAMP_OUT renamed OPAMP_OUT_LP
- net OPAMP_OUT_1 renamed TIA-OUT
- net TIA-OUT: now also C6.1, R2.1
- new net: R10.2, R9.1, U4.2 (-)
- new net: C6.2, R8.2, U4.3 (+)
- new net: C4.1, C5.1, R2.2
- new net: C4.2, R7.1, U3.2 (-)
- new net: R11.1, R9.2, U4.6
- new net OPAMP_OUT_BPF: C5.2, R7.2, U3.6
- new net OPAMP_OUT_BPF_1st: C7.2, R11.2
- new net Vref: C8.1, R12.2, R13.1, U1.3 (+)
- new net Vref_Ideal: C2.1, C7.1, R10.1, R5.1, R8.1, U3.3 (+), V5.1
- no-connect marks 4 -> 8
Other:
- moved on the sheet: C2, R4, R5, R6, U2

Commit message: Backup
Parts:
- removed C1: 2.7p, symbol Device:C
- removed C2, C7: 330p, symbol Device:C
- removed C3: 30p, symbol Device:C
- removed C4, C5: 10p, symbol Device:C
- removed C6: 1n, symbol Device:C
- removed C8: 10uF, symbol Device:C_Polarized
- removed I1: ITRNOISE, symbol Simulation_SPICE:ITRNOISE
- removed I2: AC 1 PULSE(0 4u 1n 1n 1n 0.5u 1u), symbol Simulation_SPICE:IDC
- removed R1: 82.5k, symbol Device:R
- removed R10, R5: 162, symbol Device:R
- removed R11, R6: 487, symbol Device:R
- removed R12, R13: 47k, symbol Device:R
- removed R2: 8k, symbol Device:R
- removed R3: 5G, symbol Device:R
- removed R4, R9: 825, symbol Device:R
- removed R7: 63.5k, symbol Device:R
- removed R8: 360, symbol Device:R
- removed U1, U2, U3, U4: AD8656 (1/2 equivalent), symbol Amplifier_Operational:AD8655
- removed V1: 5, symbol Simulation_SPICE:VDC
- removed V2: -5, symbol Simulation_SPICE:VDC
- removed V3: -2.75, symbol Simulation_SPICE:VDC
- removed V4: 2.75, symbol Simulation_SPICE:VDC
- removed V5: 2.5, symbol Simulation_SPICE:VDC
Connections:
- no-connect marks 8 -> 0
Other:
- added sheet Didital (digital.kicad_sch)
- added sheet Power (power.kicad_sch)
- added sheet RX frontend (receiver_analog.kicad_sch)
- added sheet TX frontend (transmitter_analog.kicad_sch)
- note removed: "SPICE photodiode equivalent"
- note removed: "Simulation DC sources"

Commit message: Laserboard backup
Other:
- sheet TX frontend ports: added AM_EN, DM_EN, TX_D_IN; removed none
Changed lines of the file:
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@@
+			)
+		)
+		(pin "AM_EN" input
+			(at 82.55 110.49 90)
+			(effects
+				(font
+					(size 1.27 1.27)
+				)
+				(justify right)
+			)
+		)
+		(pin "DM_EN" input
+			(at 85.09 110.49 90)
+			(effects
+				(font
+					(size 1.27 1.27)
+				)
+				(justify right)
+			)
+		)
+		(pin "TX_D_IN" input
+			(at 97.79 118.11 0)
+			(effects
+				(font
+					(size 1.27 1.27)
+				)
+				(justify right)
 			)
 		)

Commit message: Pre-PCB backup
Connections:
- no-connect marks 0 -> 3
Other:
- sheet Didital ports: added RX_BPF, RX_CLK, RX_CS, RX_DIO, RX_IN, RX_TIA, TX_D_IN, USB_D+, USB_D-; removed none
- sheet Power ports: added MCU_USB_D+, MCU_USB_D-; removed none
