File: laserboard/digital.kicad_sch (KiCad schematic)
At the start: 0 parts

Commit message: Laserboard backup
Parts:
- added C15, C16: 15p, Capacitor_SMD:C_0402_1005Metric, symbol Device:C
- added C19, C21, C22, C24, C26, C27, C28, C29, C30, C31: 100n, Capacitor_SMD:C_0402_1005Metric, symbol Device:C
- added C23, C25: 1u, Capacitor_SMD:C_0402_1005Metric, symbol Device:C
- added C32: 10u, Capacitor_SMD:C_0805_2012Metric, symbol Device:C
- added H1, H2, H3, H4: MountingHole, MountingHole:MountingHole_2.7mm_M2.5, symbol Mechanical:MountingHole
- added J1: Conn_01x02, Connector_PinHeader_2.54mm:PinHeader_1x02_P2.54mm_Vertical, symbol Connector_Generic:Conn_01x02
- added J3, J4: Conn_02x18_Odd_Even, Connector_PinHeader_2.54mm:PinHeader_2x18_P2.54mm_Vertical, symbol Connector_Generic:Conn_02x18_Odd_Even
- added R16, R18: 1k, Resistor_SMD:R_0402_1005Metric, symbol Device:R
- added R17: DNF, Resistor_SMD:R_0402_1005Metric, symbol Device:R
- added R19, R20: 27, Resistor_SMD:R_0402_1005Metric, symbol Device:R
- added U6: W25Q128JVS, Package_SO:SOIC-8_5.23x5.23mm_P1.27mm, symbol Memory_Flash:W25Q128JVS
- added U7: RP2040, RP2040_minimal:RP2040-QFN-56, symbol MCU_RaspberryPi_RP2040:RP2040
- added Y1: ABM8-272-T3, Crystal:Crystal_SMD_3225-4Pin_3.2x2.5mm, symbol Device:Crystal_GND24
Connections:
- new net: C16.1, R18.2, Y1.3
- new net: R20.2, U7.46 (USB_DM)
- new net: R19.2, U7.47 (USB_DP)
- new net +1V1: C21.1, C22.1, C23.1, U7.23 (DVDD), U7.45 (VREG_VOUT), U7.50 (DVDD)
- new net +3V3: C19.1, C24.1, C25.1, C26.1, C27.1, C28.1, C29.1, C30.1, C31.1, C32.1, J3.2 (Pin_2), R17.1, U6.8 (VCC), U7.1 (IOVDD), U7.10 (IOVDD), U7.22 (IOVDD), U7.33 (IOVDD), U7.42 (IOVDD), U7.43 (ADC_AVDD), U7.44 (VREG_IN), U7.48 (USB_VDD), U7.49 (IOVDD)
- new net GND: C15.2, C16.2, C19.2, C21.2, C22.2, C23.2, C24.2, C25.2, C26.2, C27.2, C28.2, C29.2, C30.2, C31.2, C32.2, J1.2 (Pin_2), J3.1 (Pin_1), J3.11 (Pin_11), J3.13 (Pin_13), J3.15 (Pin_15), J3.17 (Pin_17), J3.19 (Pin_19), J3.21 (Pin_21), J3.23 (Pin_23), J3.25 (Pin_25), J3.27 (Pin_27), J3.29 (Pin_29), J3.3 (Pin_3), J3.31 (Pin_31), J3.33 (Pin_33), J3.35 (Pin_35), J3.36 (Pin_36), J3.5 (Pin_5), J3.7 (Pin_7), J3.9 (Pin_9), J4.10 (Pin_10), J4.12 (Pin_12), J4.14 (Pin_14), J4.16 (Pin_16), J4.18 (Pin_18), J4.2 (Pin_2), J4.20 (Pin_20), J4.22 (Pin_22), J4.24 (Pin_24), J4.26 (Pin_26), J4.28 (Pin_28), J4.30 (Pin_30), J4.32 (Pin_32), J4.34 (Pin_34), J4.35 (Pin_35), J4.36 (Pin_36), J4.4 (Pin_4), J4.6 (Pin_6), J4.8 (Pin_8), U6.4 (GND), U7.19 (TESTEN), U7.57 (GND), Y1.2, Y1.4
- new net GPIO0: J3.4 (Pin_4), U7.2 (GPIO0)
- new net GPIO1: J3.6 (Pin_6), U7.3 (GPIO1)
- new net GPIO10: J3.24 (Pin_24), U7.13 (GPIO10)
- new net GPIO11: J3.26 (Pin_26), U7.14 (GPIO11)
- new net GPIO12: J3.28 (Pin_28), U7.15 (GPIO12)
- new net GPIO13: J3.30 (Pin_30), U7.16 (GPIO13)
- new net GPIO14: J3.32 (Pin_32), U7.17 (GPIO14)
- new net GPIO15: J3.34 (Pin_34), U7.18 (GPIO15)
- new net GPIO16: J4.27 (Pin_27), U7.27 (GPIO16)
- new net GPIO17: J4.25 (Pin_25), U7.28 (GPIO17)
- new net GPIO18: J4.23 (Pin_23), U7.29 (GPIO18)
- new net GPIO19: J4.21 (Pin_21), U7.30 (GPIO19)
- new net GPIO2: J3.8 (Pin_8), U7.4 (GPIO2)
- new net GPIO20: J4.19 (Pin_19), U7.31 (GPIO20)
- new net GPIO21: J4.17 (Pin_17), U7.32 (GPIO21)
- new net GPIO22: J4.15 (Pin_15), U7.34 (GPIO22)
- new net GPIO23: J4.13 (Pin_13), U7.35 (GPIO23)
- new net GPIO24: J4.11 (Pin_11), U7.36 (GPIO24)
- new net GPIO25: J4.9 (Pin_9), U7.37 (GPIO25)
- new net GPIO26_ADC0: J4.7 (Pin_7), U7.38 (GPIO26_ADC0)
- new net GPIO27_ADC1: J4.5 (Pin_5), U7.39 (GPIO27_ADC1)
- new net GPIO28_ADC2: J4.3 (Pin_3), U7.40 (GPIO28_ADC2)
- new net GPIO29_ADC3: J4.1 (Pin_1), U7.41 (GPIO29_ADC3)
- new net GPIO3: J3.10 (Pin_10), U7.5 (GPIO3)
- new net GPIO4: J3.12 (Pin_12), U7.6 (GPIO4)
- new net GPIO5: J3.14 (Pin_14), U7.7 (GPIO5)
- new net GPIO6: J3.16 (Pin_16), U7.8 (GPIO6)
- new net GPIO7: J3.18 (Pin_18), U7.9 (GPIO7)
- new net GPIO8: J3.20 (Pin_20), U7.11 (GPIO8)
- new net GPIO9: J3.22 (Pin_22), U7.12 (GPIO9)
- new net QSPI_SCLK: U6.6 (CLK), U7.52 (QSPI_SCLK)
- new net QSPI_SD0: U6.5 (DI(IO0)), U7.53 (QSPI_SD0)
- new net QSPI_SD1: U6.2 (DO(IO1)), U7.55 (QSPI_SD1)
- new net QSPI_SD2: U6.3 (IO2), U7.54 (QSPI_SD2)
- new net QSPI_SD3: U6.7 (IO3), U7.51 (QSPI_SD3)
- new net QSPI_SS: R16.1, R17.2, U6.1 (~{CS}), U7.56 (QSPI_SS)
- new net RUN: J4.29 (Pin_29), U7.26 (RUN)
- new net SWCLK: J4.33 (Pin_33), U7.24 (SWCLK)
- new net SWD: J4.31 (Pin_31), U7.25 (SWD)
- new net USB_D+: R19.1
- new net USB_D-: R20.1
- new net XIN: C15.1, U7.20 (XIN), Y1.1
- new net XOUT: R18.1, U7.21 (XOUT)
- new net ~{USB_BOOT}: J1.1 (Pin_1), R16.2
Other:
- note added: "Crystal"
- note added: "Flash"
- note added: "IOs"
- note added: "Make sure 19 and R20 are close to RP2040"
- note added: "Make sure C23 is close to pin 45 of RP2040"
- note added: "Make sure C25 is close to pin 44 of RP2040"

Commit message: Backup
Parts:
- removed J3: Conn_02x18_Odd_Even, Connector_PinHeader_2.54mm:PinHeader_2x18_P2.54mm_Vertical, symbol Connector_Generic:Conn_02x18_Odd_Even
- added D3: LED, symbol Device:LED
- added J3: Conn_01x19, Connector_PinHeader_2.54mm:PinHeader_1x19_P2.54mm_Vertical, symbol Connector_Generic:Conn_01x19
- added JP6: SolderJumper_2_Open, Jumper:SolderJumper-2_P1.3mm_Open_Pad1.0x1.5mm, symbol Jumper:SolderJumper_2_Open
- J4: value Conn_02x18_Odd_Even -> Conn_01x19; footprint Connector_PinHeader_2.54mm:PinHeader_2x18_P2.54mm_Vertical -> Connector_PinHeader_2.54mm:PinHeader_1x19_P2.54mm_Vertical; symbol Connector_Generic:Conn_02x18_Odd_Even -> Connector_Generic:Conn_01x19
- R17: now not fitted
Connections:
- net +3V3: now also J3.18 (Pin_18)
- net GND: now also J4.1 (Pin_1), J4.19 (Pin_19), J3.1 (Pin_1); no longer J4.10 (Pin_10), J4.12 (Pin_12), J4.14 (Pin_14), J4.16 (Pin_16), J4.18 (Pin_18), J4.2 (Pin_2), J4.20 (Pin_20), J4.22 (Pin_22), J4.24 (Pin_24), J4.26 (Pin_26), J4.28 (Pin_28), J4.30 (Pin_30), J4.32 (Pin_32), J4.34 (Pin_34), J4.35 (Pin_35), J4.36 (Pin_36), J4.4 (Pin_4), J4.6 (Pin_6), J4.8 (Pin_8)
- net GPIO1: now also J3.16 (Pin_16)
- net GPIO10: now also J3.7 (Pin_7)
- net GPIO11: now also J3.6 (Pin_6)
- net GPIO12: now also J3.5 (Pin_5)
- net GPIO13: now also J3.4 (Pin_4)
- net GPIO14: now also J3.3 (Pin_3)
- net GPIO15: now also J3.2 (Pin_2)
- net GPIO16: now also J4.15 (Pin_15); no longer J4.27 (Pin_27)
- net GPIO2: now also J3.15 (Pin_15)
- net GPIO20: now also J4.11 (Pin_11); no longer J4.19 (Pin_19)
- net GPIO21: now also J4.10 (Pin_10); no longer J4.17 (Pin_17)
- net GPIO22: now also J4.9 (Pin_9); no longer J4.15 (Pin_15)
- net GPIO23: now also J4.8 (Pin_8); no longer J4.13 (Pin_13)
- net GPIO24: now also J4.7 (Pin_7); no longer J4.11 (Pin_11)
- net GPIO25: now also J4.6 (Pin_6); no longer J4.9 (Pin_9)
- net GPIO26_ADC0: now also J4.5 (Pin_5), JP6.2 (B); no longer J4.7 (Pin_7), U7.38 (GPIO26_ADC0)
- net GPIO29_ADC3: now also J4.2 (Pin_2); no longer J4.1 (Pin_1)
- net GPIO3: now also J3.14 (Pin_14)
- net GPIO4: now also J3.13 (Pin_13)
- net GPIO5: now also J3.12 (Pin_12)
- net GPIO6: now also J3.11 (Pin_11)
- net GPIO7: now also J3.10 (Pin_10)
- net GPIO8: now also J3.9 (Pin_9)
- net GPIO9: now also J3.8 (Pin_8)
- net RUN: now also J4.16 (Pin_16); no longer J4.29 (Pin_29)
- net SWCLK: now also J4.18 (Pin_18); no longer J4.33 (Pin_33)
- net SWD: now also J4.17 (Pin_17); no longer J4.31 (Pin_31)
- net GPIO0 renamed TX_D_IN
- net TX_D_IN: now also J3.17 (Pin_17)
- net GPIO17 renamed RX_CS
- net RX_CS: now also J4.14 (Pin_14); no longer J4.25 (Pin_25)
- net GPIO18 renamed RX_CLK
- net RX_CLK: now also J4.13 (Pin_13); no longer J4.23 (Pin_23)
- net GPIO19 renamed RX_DIO
- net RX_DIO: now also J4.12 (Pin_12); no longer J4.21 (Pin_21)
- net GPIO27_ADC1 renamed RX_BPF
- net RX_BPF: now also J4.4 (Pin_4); no longer J4.5 (Pin_5)
- net GPIO28_ADC2 renamed RX_TIA
- new net RX_IN: JP6.1 (A), U7.38 (GPIO26_ADC0)
- new net VBUS: J3.19 (Pin_19)
Other:
- note added: "Do I want output on the ADC0 pin or the cleanest measurement for MCU?"
- note added: "IO connectors will not be placed by default"

Commit message: Pre-PCB backup
Parts:
- added D4: LED, LED_SMD:LED_0603_1608Metric, symbol Device:LED
- added R28, R30: 220, Resistor_SMD:R_0402_1005Metric, symbol Device:R
- D3: footprint (none) -> LED_SMD:LED_0603_1608Metric
- U6: footprint Package_SO:SOIC-8_5.23x5.23mm_P1.27mm -> Package_SO:SOIC-8_5.3x5.3mm_P1.27mm
Connections:
- net GND: now also D3.1 (K), D4.1 (K)
- net GPIO24: now also R30.2
- net GPIO25: now also R28.2
- net at D3.2 (A): now also R28.1
- new net: D4.2 (A), R30.1
Other:
- moved on the sheet: D3, JP6

Commit message: AF PCB stage backup
Parts:
- R28, R30: value 220 -> 470
Changed lines of the file:
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@@
 			)
 		)
-		(property "Value" "220"
+		(property "Value" "470"
 			(at 223.52 124.0536 90)
 			(effects
@@
 			)
 		)
-		(property "Value" "220"
+		(property "Value" "470"
 			(at 223.52 131.6736 90)
 			(effects

Commit message: PCB_prot
Parts:
- added JP8: SolderJumper_2_Open, Jumper:SolderJumper-2_P1.3mm_Open_Pad1.0x1.5mm, symbol Jumper:SolderJumper_2_Open
Connections:
- net GND: now also J4.16 (Pin_16), J4.17 (Pin_17), J4.18 (Pin_18)
- net GPIO10: now also R28.2
- net GPIO11: now also R30.2
- net GPIO15: now also JP8.2 (B); no longer U7.18 (GPIO15)
- net GPIO16: now also J4.12 (Pin_12); no longer J4.15 (Pin_15)
- net GPIO24: no longer R30.2
- net GPIO25: no longer R28.2
- net RUN: now also J4.13 (Pin_13); no longer J4.16 (Pin_16)
- net RX_CLK: no longer J4.13 (Pin_13)
- net RX_CS: no longer J4.14 (Pin_14)
- net RX_DIO: no longer J4.12 (Pin_12)
- net SWCLK: now also J4.15 (Pin_15); no longer J4.18 (Pin_18)
- net SWD: now also J4.14 (Pin_14); no longer J4.17 (Pin_17)
- net TX_D_IN: now also U7.18 (GPIO15), JP8.1 (A); no longer J3.17 (Pin_17), U7.2 (GPIO0)
- new net GPIO0: J3.17 (Pin_17), U7.2 (GPIO0)
Other:
- moved on the sheet: D3, D4, R28, R30

Commit message: Post-production commit
Parts:
- C15, C16, C19, C21, C22, C23, C24, C25, C26, C27, C28, C29, C30, C31: footprint Capacitor_SMD:C_0402_1005Metric -> parts:C_0402_1005Metric_nosilk
- R16, R17, R18, R19, R20, R28, R30: footprint Resistor_SMD:R_0402_1005Metric -> parts:R_0402_1005Metric_nosilk
