File: laserboard/receiver_analog.kicad_sch (KiCad schematic)
At the start: 31 parts, among them U1 AD8656, U2 PGA112, U3 AD8655, U4 LM4040DBZ-2.5

Commit message: Update
Parts:
- added C20: 10n, symbol Device:C
- added R29: 1.6M, symbol Device:R
Connections:
- net GND: now also R29.1
- net at C3.1, R1.1, U3.2 (-): now also C20.1; no longer JP2.2 (B)
- net at D1.2 (A), JP1.1 (A): now also JP2.2 (B); no longer JP2.1 (A)
- new net: C20.2, JP2.1 (A), R29.2
Other:
- moved on the sheet: JP1, JP2

Commit message: Laserboard backup
Changed lines of the file:
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@@
 	(wire
 		(pts
-			(xy 39.37 48.26) (xy 39.37 55.88)
+			(xy 39.37 48.26) (xy 39.37 66.04)
 		)
 		(stroke
@@
 	)
 	(label "Vref_Filter"
-		(at 39.37 55.88 180)
+		(at 39.37 66.04 180)
 		(effects
 			(font
@@
 		(dnp no)
 		(property "Reference" "C20"
-			(at 33.528 64.516 0)
-			(effects
-				(font
-					(size 1.27 1.27)
-				)
-				(hide yes)
-			)
-		)
+			(at 25.908 55.118 90)
+			(effects
+				(font
+					(size 1.27 1.27)
+				)
+			)
+		)

Commit message: Update
Parts:
- added C33: 4.7uF, symbol Device:C_Polarized
- added C34: 100p, symbol Device:C
- added R23, R24: 220k, symbol Device:R
- added R25, R26: RSHUNT_BACKUP, symbol Device:R
- C10, C9, TP3, U4: now not fitted; now left out of the parts list
- R7: now not fitted
Connections:
- net +3V3: now also C2.2, D1.1 (K), U1.8 (V+), U2.1 (AV_{DD}), U3.7 (V+), R23.2, R25.1
- net +5V: no longer C2.2, D1.1 (K), U1.8 (V+), U2.1 (AV_{DD}), U3.7 (V+)
- net GND: now also C33.2, C34.2, R24.1, R26.2
- net RX_Raw: no longer U2.3 (CH0/V_{CAL})
- net Vref_Filter: now also C33.1, C34.1, R23.1, R24.2, R25.2, R26.1
- no-connect marks 2 -> 3
Other:
- note removed: "MAX - 4-4.5 mA for the circuit"

Commit message: Backup
Parts:
- JP1: now not fitted
Changed lines of the file:
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@@
 	(generator_version "9.0")
 	(paper "A4")
+	(text_box "RX reception + filtration + amplification. \nFilter is designed to bandpass 300kHz to 1MHz. Also it blocks DC light. \nPGA amplifier can be used to control the gain and increase SNR of the signal.\nFor testing, testpoints are available. \nFor external analysis, outputs are traced* to the connectors (connect solderjumpers for this)\n* - connected hardware can change frequency characteristics of the frontend"
+		(exclude_from_sim no)
+		(at 217.17 17.78 0)
+		(size 66.04 48.26)
+		(margins 0.9525 0.9525 0.9525 0.9525)
+		(stroke
+			(width 0)
+			(type solid)
+		)
+		(fill
+			(type none)
+		)
+		(effects
+			(font
+				(size 1.27 1.27)
+			)
+			(justify left top)
+		)
+	)
 	(junction
 		(at 160.02 95.25)
@@
 		(exclude_from_sim no)
 		(in_bom no)
-		(on_board yes)
-		(dnp no)
+		(on_board no)
+		(dnp yes)
 		(property "Reference" "JP1"
 			(at 13.716 42.164 90)

Commit message: Pre-PCB backup
Parts:
- added C35, C37: 0.1uF, Capacitor_SMD:C_0402_1005Metric, symbol Device:C
- added C36: 4.7uF, Capacitor_Tantalum_SMD:CP_EIA-2012-12_Kemet-R_HandSolder, symbol Device:C_Polarized
- C1, C2, C3, C34, C4, C5, C6, C7, C8: footprint (none) -> Capacitor_SMD:C_0402_1005Metric
- C33: footprint (none) -> Capacitor_Tantalum_SMD:CP_EIA-2012-12_Kemet-R_HandSolder
- R1, R2, R3, R4, R5, R6, R8: footprint (none) -> Resistor_SMD:R_0402_1005Metric
- R23, R24, R25, R26: footprint (none) -> Resistor_SMD:R_0805_2012Metric_Pad1.20x1.40mm_HandSolder
- U1, U3: footprint (none) -> Package_SO:SOIC-8_3.9x4.9mm_P1.27mm
Connections:
- net +3V3: now also C35.1, C36.1, C37.1
- net GND: now also C35.2, C36.2, C37.2

Commit message: AF PCB stage backup
Parts:
- C20: footprint (none) -> Capacitor_SMD:C_0402_1005Metric; now in the parts list
- R29: footprint (none) -> Resistor_SMD:R_0805_2012Metric; now in the parts list
Changed lines of the file:
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@@
 		(unit 1)
 		(exclude_from_sim no)
-		(in_bom no)
-		(on_board no)
+		(in_bom yes)
+		(on_board yes)
 		(dnp no)
 		(property "Reference" "C20"
@@
 			)
 		)
-		(property "Footprint" ""
+		(property "Footprint" "Capacitor_SMD:C_0402_1005Metric"
 			(at 22.86 61.9252 0)
 			(effects
@@
 		(unit 1)
 		(exclude_from_sim no)
-		(in_bom no)
-		(on_board no)
+		(in_bom yes)
+		(on_board yes)
 		(dnp no)
 		(property "Reference" "R29"
@@
 			)
 		)
-		(property "Footprint" ""
+		(property "Footprint" "Resistor_SMD:R_0805_2012Metric"
 			(at 23.368 64.77 90)
 			(effects

Commit message: PCB_prot
Parts:
- JP3, JP4: now not fitted
Changed lines of the file:
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@@
 		(exclude_from_sim no)
 		(in_bom no)
-		(on_board yes)
-		(dnp no)
+		(on_board no)
+		(dnp yes)
 		(fields_autoplaced yes)
 		(property "Reference" "JP3"
@@
 		(exclude_from_sim no)
 		(in_bom no)
-		(on_board yes)
-		(dnp no)
+		(on_board no)
+		(dnp yes)
 		(fields_autoplaced yes)
 		(property "Reference" "JP4"

Commit message: Post-production commit
Parts:
- C1, C2, C20, C3, C34, C35, C4, C5, C6, C7, C8: footprint Capacitor_SMD:C_0402_1005Metric -> parts:C_0402_1005Metric_nosilk
- R1, R2, R3, R4, R5, R6, R8: footprint Resistor_SMD:R_0402_1005Metric -> parts:R_0402_1005Metric_nosilk
